Commit message: connected ui to bot

File: bot/public/model/arm.urdf (robot description, URDF)
Before this commit: robot V0.01, 19 links, 18 joints
Joints:
- joint 2-clamp_Rigid-5: origin xyz=0.02860641 0.043999999999999984 0.004505069999999996 rpy=3.5437110976725134e-32 -1.5707963267948966 0 -> xyz=0.02535 0.044 -0.014000000000000002 rpy=1.7791258877055312e-34 -1.5707963267948966 0
- joint 2-holder_Rigid-4: origin xyz=-0.0424048 0.03296393 0.0123 rpy=1.5707963267948966 2.0029671421627253e-32 -5.551115123125783e-17 -> xyz=-0.05371022 0.0 0.0123 rpy=1.5707963267948966 4.3608013207788786e-33 6.162975822039155e-33
- joint 2-servo_2-pitch: axis -0.613737 1.7530665807896634e-16 0.789511 -> 1.9721522630525295e-31 2.220446049250313e-16 1.0; origin xyz=0.02459326 -0.012999999999999989 0.019117899999999993 rpy=2.220446049250313e-16 1.5707963267948966 0 -> xyz=0.031150000000000004 -0.012999999999999989 0.0 rpy=2.220446049250313e-16 1.5707963267948966 0
- joint 3-clamp_Rigid-8: origin xyz=0.043330780000000006 -0.02535 0.015951260000000002 rpy=4.379057701015054e-47 -1.5707963267948966 0 -> xyz=0.044000000000000004 -0.02535 -0.013999999999999999 rpy=-5.470005157845276e-31 -1.5707963267948966 0
- joint 3-holder_Rigid-7: origin xyz=0.030064509999999992 0.16658488999999999 0.0006987699999999652 rpy=-2.775557561562891e-16 -5.551115123125743e-17 4.067564042545841e-31 -> xyz=0.02416511 0.16658488999999999 -0.01790000000000004 rpy=-2.220446049250313e-16 1.972152263052531e-31 5.261630935975519e-31
- joint 3-servo_3-pitch: axis -0.613737 1.7530665807896658e-16 0.7895109999999997 -> 3.944304526105059e-31 2.220446049250313e-16 1.0; origin xyz=0.016614689999999994 0.0 0.029381530000000003 rpy=2.220446049250313e-16 1.5707963267948966 0 -> xyz=0.031150000000000004 0.0 0.013000000000000003 rpy=2.2204460492503136e-16 1.5707963267948966 0
- joint 4-clamp_Rigid-11: origin xyz=0.04333079 -0.02535 -0.015951260000000005 rpy=1.5707963267948966 5.551115123125783e-17 3.944304526105059e-31 -> xyz=0.044000000000000004 -0.02535 0.013999999999999999 rpy=1.5707963267948966 3.944304526105059e-31 -3.257879004812441e-31
- joint 4-holder_Rigid-10: origin xyz=0.10566016000000002 -0.026034889999999998 0.059464050000000025 rpy=3.141592653589793 -7.88860905221012e-31 3.944304526105062e-31 -> xyz=0.11991510999999999 -0.026034889999999998 -0.017899999999999996 rpy=3.141592653589793 3.944304526105061e-31 9.04679294230822e-31
- joint 4-servo_4-pitch: axis 0.6137369999999999 -1.3411034749590469e-31 0.789511 -> -3.944304526105059e-31 7.395570986446986e-31 1.0; origin xyz=-0.006734650000000002 0.012518259999999995 0.0 rpy=-1.5707963267948966 -1.5777218104420234e-30 -1.2325951644078312e-32 -> xyz=-0.013000000000000008 0.00575 0.0 rpy=-1.5707963267948966 4.721721744173088e-31 0.0
- joint 5-clamp_Rigid-14: origin xyz=0.04333078999999998 -0.02535 0.015951260000000005 rpy=-1.5707963267948966 1.5707963267948966 0 -> xyz=0.044000000000000004 -0.02535 -0.013999999999999986 rpy=-1.5707963267948966 1.5707963267948966 0
- joint 5-holder_Rigid-13: origin xyz=0.040961809999999994 -0.02575000000000003 -0.021899339999999993 rpy=3.141592653589793 1.5707963267948963 0 -> xyz=0.04578022000000001 -0.025749999999999995 0.007850000000000001 rpy=3.141592653589793 1.5707963267948963 0
- joint 5-servo_5-roll: axis 0.6137369999999999 1.753066580789639e-16 0.789511 -> 0.0 2.2204460492502372e-16 1.0; origin xyz=0.012518270000000022 0.0067346599999999765 0.0 rpy=-1.5707963267948963 4.7331654313260715e-30 -1.5707963267948968 -> xyz=0.0057500000000000285 0.013000000000000001 0.0 rpy=-1.5707963267948963 3.1554436208840472e-30 -1.5707963267948966
- joint 6-clamp_Rigid-17: origin xyz=0.019180250000000003 -0.014000000000000021 0.04701851 rpy=-1.5707963267948966 -3.1554436208840472e-30 0.0 -> xyz=0.044000000000000025 -0.014000000000000021 0.02535 rpy=-1.5707963267948966 -1.2347103262258056e-30 1.9480294112644395e-60
- joint 6-holder_Rigid-16: origin xyz=-0.013621080000000028 0.029349999999999987 0.025110320000000002 rpy=3.141592653589793 -1.5707963267948963 0 -> xyz=-0.026165110000000002 0.029350000000000022 0.011465119999999978 rpy=3.141592653589793 -1.5707963267948963 0
- joint 6-servo_6-grip: axis -0.0 1.0 -2.220446049250345e-16 -> -0.0 1.0 -2.2204460492503136e-16; origin xyz=-0.01026364000000001 0.007978570000000004 -0.005749999999999993 rpy=-1.5707963267948963 -0.0 0.0 -> xyz=-0.013000000000000008 0.0 -0.005749999999999993 rpy=-1.5707963267948963 3.4702805965586234e-60 -2.1995516405939585e-30
